File: PCB/coaster.kicad_pcb (KiCad board)
At the start: 2 copper layers, 65 x 70 mm, 83 parts, among them J1 AVR-ISP-6, J10 Conn_01x04, J11 Barrel_Jack, J2 USB_B_Micro, J3 Conn_01x02, J4 Conn_01x02, J5 Conn_01x02, J6 Conn_01x03, J7 Conn_01x03, J8 Conn_01x04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

Commit message: cleaned in pcb
Parts:
- C23, C26, C27, C28, C30: value 0.1u -> 100n
- C29: value C -> 100n
- R10, R4, R6, R8: value R -> 100
- R11, R12, R13, R5, R7, R9: value R -> 120
- Y1: value ECS-160-12-33-AGN-TR -> 16MHz 12pF 60 Ohm +/- 10 ppm
Connections:
- J2 pad 1: Net-(FB1-Pad2) -> unconnected-(J2-Pad1)
