File: PCB/coaster.kicad_sch (KiCad schematic)
At the start: 84 parts, among them J1 AVR-ISP-6, J10 Conn_01x04, J11 Barrel_Jack, J2 USB_B_Micro, J3 Conn_01x02, J4 Conn_01x02, J5 Conn_01x02, J6 Conn_01x03, J7 Conn_01x03, J8 Conn_01x04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

Commit message: cleaned in pcb
Parts:
- removed FB1: FerriteBead, Resistor_SMD:R_1206_3216Metric_Pad1.30x1.75mm_HandSolder, symbol Device:FerriteBead
- C1, C10, C11, C12, C13, C14, C15, C2, C3, C7, C8, C9: value 100n -> (none); footprint Capacitor_SMD:C_1206_3216Metric_Pad1.33x1.80mm_HandSolder -> (none); LCSC (none) -> C24497
- C16, C17, C18: value 22n -> (none); footprint Capacitor_SMD:C_1206_3216Metric_Pad1.33x1.80mm_HandSolder -> (none); LCSC (none) -> C113907
- C19, C20, C21: value 2.2u -> (none); footprint Capacitor_SMD:C_1206_3216Metric_Pad1.33x1.80mm_HandSolder -> (none); LCSC (none) -> C50254
- C22: value 0.33u -> (none); footprint Capacitor_SMD:C_1206_3216Metric_Pad1.33x1.80mm_HandSolder -> (none); LCSC (none) -> C307572
- C23, C26, C27, C28, C29, C30: value 0.1u -> (none); footprint Capacitor_SMD:C_1206_3216Metric_Pad1.33x1.80mm_HandSolder -> (none); LCSC (none) -> C24497
- C24, C25: value 20p -> (none); footprint Capacitor_SMD:C_1206_3216Metric_Pad1.33x1.80mm_HandSolder -> (none); LCSC (none) -> C162447
- C4, C5, C6: value 100u -> (none); footprint Capacitor_SMD:CP_Elec_5x5.4 -> (none); LCSC (none) -> C487302
- D1: value M1EN -> (none); footprint LED_SMD:LED_1206_3216Metric_Pad1.42x1.75mm_HandSolder -> (none); LCSC (none) -> C84273
- D10, D8, D9: value LED -> (none); footprint LED_SMD:LED_1206_3216Metric_Pad1.42x1.75mm_HandSolder -> (none); LCSC (none) -> C93133
- D2: value M1STEP -> (none); footprint LED_SMD:LED_1206_3216Metric_Pad1.42x1.75mm_HandSolder -> (none); LCSC (none) -> C93133
- D3: value M2EN -> (none); footprint LED_SMD:LED_1206_3216Metric_Pad1.42x1.75mm_HandSolder -> (none); LCSC (none) -> C84273
- D4: value M2STEP -> (none); footprint LED_SMD:LED_1206_3216Metric_Pad1.42x1.75mm_HandSolder -> (none); LCSC (none) -> C93133
- D5: value M3EN -> (none); footprint LED_SMD:LED_1206_3216Metric_Pad1.42x1.75mm_HandSolder -> (none); LCSC (none) -> C84273
- D6: value M3STEP -> (none); footprint LED_SMD:LED_1206_3216Metric_Pad1.42x1.75mm_HandSolder -> (none); LCSC (none) -> C93133
- D7: value PWR -> (none); footprint LED_SMD:LED_1206_3216Metric_Pad1.42x1.75mm_HandSolder -> (none); LCSC (none) -> C84273
- FB2: value FerriteBead -> (none); footprint Resistor_SMD:R_1206_3216Metric_Pad1.30x1.75mm_HandSolder -> (none); LCSC (none) -> C139169
- J1: value AVR-ISP-6 -> (none); footprint Connector_PinHeader_2.54mm:PinHeader_2x03_P2.54mm_Vertical -> (none)
- J10, J8, J9: value Conn_01x04 -> (none); footprint Connector_JST:JST_XH_B4B-XH-A_1x04_P2.50mm_Vertical -> (none)
- J11: value Barrel_Jack -> (none); footprint Connector_BarrelJack:BarrelJack_Horizontal -> (none)
- J2: value USB_B_Micro -> (none); footprint Connector_USB:USB_Micro-B_Amphenol_10104110_Horizontal -> (none)
- J3, J4, J5: value Conn_01x02 -> (none); footprint Connector_JST:JST_XH_B2B-XH-A_1x02_P2.50mm_Vertical -> (none)
- J6, J7: value Conn_01x03 -> (none); footprint Connector_JST:JST_XH_B3B-XH-A_1x03_P2.50mm_Vertical -> (none)
- R1, R2: value 1k -> (none); footprint Resistor_SMD:R_1206_3216Metric_Pad1.30x1.75mm_HandSolder -> (none); LCSC (none) -> C4410
- R10, R4, R6, R8: value 100 -> (none); footprint Resistor_SMD:R_1206_3216Metric_Pad1.30x1.75mm_HandSolder -> (none); LCSC (none) -> C17901
- R11, R12, R13, R5, R7, R9: value 120 -> (none); footprint Resistor_SMD:R_1206_3216Metric_Pad1.30x1.75mm_HandSolder -> (none); LCSC (none) -> C17909
- R14, R15, R16, R3: value 10k -> (none); footprint Resistor_SMD:R_1206_3216Metric_Pad1.30x1.75mm_HandSolder -> (none); LCSC (none) -> C17902
- R17, R18: value 22 -> (none); footprint Resistor_SMD:R_1206_3216Metric_Pad1.30x1.75mm_HandSolder -> (none); LCSC (none) -> C5672
- R19, R20, R21, R22: value 0 -> (none); footprint Resistor_SMD:R_1206_3216Metric_Pad1.30x1.75mm_HandSolder -> (none); LCSC (none) -> C17888
- RV1, RV2: value CG0603MLC-05E -> (none); footprint Resistor_SMD:R_0603_1608Metric_Pad0.98x0.95mm_HandSolder -> (none); LCSC (none) -> C20960
- U1, U2, U3: value TMC2208-LA -> (none); footprint TMC2208:TMC2208-LA -> (none); LCSC (none) -> C115944
- U4: value uA7805 -> (none); footprint Package_TO_SOT_SMD:SOT-89-3_Handsoldering -> (none); LCSC (none) -> C962135
- U5: value ATmega128-16A -> (none); footprint Package_QFP:TQFP-64_14x14mm_P0.8mm -> (none); LCSC (none) -> C183188
- U6: value CH340E -> (none); footprint Package_SO:MSOP-10_3x3mm_P0.5mm -> (none); LCSC (none) -> C99652
- Y1: footprint TMC2208:XTAL_ECS-160-12-33-AGN-TR -> (none); LCSC (none) -> C89371

Commit message: added some sourcing
Parts:
- J11: ELFA (none) -> 301-29-715
- J2: Digikey (none) -> 609-4052-1-ND; ELFA (none) -> 301-61-489
Changed lines of the file:
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@@
+      (effects (font (size 1.27 1.27)) hide)
+    )
+    (property "Digikey" "609-4052-1-ND" (id 4) (at 97.79 139.7 0)
+      (effects (font (size 1.27 1.27)) hide)
+    )
+    (property "ELFA" "301-61-489" (id 5) (at 97.79 139.7 0)
       (effects (font (size 1.27 1.27)) hide)
     )
@@
       (effects (font (size 1.27 1.27)) hide)
     )
+    (property "ELFA" "301-29-715" (id 4) (at 220.98 152.4 0)
+      (effects (font (size 1.27 1.27)) hide)
+    )
